Commit message: feat: moveit 配置与urdf路径更新

File: src/arm_description/urdf/miniarm.urdf (robot description, URDF)
Before this commit: robot mini1, 7 links, 6 joints
Links:
- link base_link: geometry collision mesh filename=package://arm_description/meshes/base_link.STL; visual mesh filename=package://arm_description/meshes/base_link.STL
- link link1: geometry collision mesh filename=package://arm_description/meshes/link1.STL; visual mesh filename=package://arm_description/meshes/link1.STL
- link link2: geometry collision mesh filename=package://arm_description/meshes/link2.STL; visual mesh filename=package://arm_description/meshes/link2.STL
- link link3: geometry collision mesh filename=package://arm_description/meshes/link3.STL; visual mesh filename=package://arm_description/meshes/link3.STL
- link link4: geometry collision mesh filename=package://arm_description/meshes/link4.STL; visual mesh filename=package://arm_description/meshes/link4.STL
- link link5: geometry collision mesh filename=package://arm_description/meshes/link5.STL; visual mesh filename=package://arm_description/meshes/link5.STL
- link link6: geometry collision mesh filename=package://arm_description/meshes/link6.STL; visual mesh filename=package://arm_description/meshes/link6.STL

File: src/arm_moveit_config/config/mini1.ros2_control.xacro (robot description, xacro)
@@ -10,4 +10,5 @@
             <joint name="joint1">
                 <command_interface name="position"/>
+                <command_interface name="velocity"/>
                 <state_interface name="position">
                   <param name="initial_value">${initial_positions['joint1']}</param>
@@ -17,4 +18,5 @@
             <joint name="joint2">
                 <command_interface name="position"/>
+                <command_interface name="velocity"/>
                 <state_interface name="position">
                   <param name="initial_value">${initial_positions['joint2']}</param>
@@ -24,4 +26,5 @@
             <joint name="joint3">
                 <command_interface name="position"/>
+                <command_interface name="velocity"/>
                 <state_interface name="position">
                   <param name="initial_value">${initial_positions['joint3']}</param>
@@ -31,4 +34,5 @@
             <joint name="joint4">
                 <command_interface name="position"/>
+                <command_interface name="velocity"/>
                 <state_interface name="position">
                   <param name="initial_value">${initial_positions['joint4']}</param>
@@ -38,4 +42,5 @@
             <joint name="joint5">
                 <command_interface name="position"/>
+                <command_interface name="velocity"/>
                 <state_interface name="position">
                   <param name="initial_value">${initial_positions['joint5']}</param>
@@ -45,4 +50,5 @@
             <joint name="joint6">
                 <command_interface name="position"/>
+                <command_interface name="velocity"/>
                 <state_interface name="position">
                   <param name="initial_value">${initial_positions['joint6']}</param>

File: src/arm_moveit_config/config/mini1.urdf.xacro (robot description, xacro)
@@ -3,5 +3,5 @@
     <xacro:arg name="initial_positions_file" default="initial_positions.yaml" />
     <!-- Import mini1 urdf file -->
-    <xacro:include filename="$(find arm_plan_node)/model/urdf/miniarm.urdf" />
+    <xacro:include filename="$(find arm_description)/urdf/miniarm.urdf" />
     <!-- Import control_xacro -->
     <xacro:include filename="mini1.ros2_control.xacro" />

Commit message: feat: (todo 修复urdf）

File: src/arm_description/urdf/miniarm.urdf (robot description, URDF)
Before this commit: robot mini1, 7 links, 6 joints
Joints:
- joint joint2: axis 0 0 -1 -> 0 0 1
- joint joint3: axis 0 0 -1 -> 0 0 1
- joint joint4: origin xyz=0 0.012 0.054 rpy=1.5708 0 3.1416 -> xyz=0 0.012 0.054 rpy=-1.5708 0 0

Commit message: feat: urdf修复完毕

File: src/arm_description/urdf/miniarm.urdf (robot description, URDF)
Before this commit: robot mini1, 7 links, 6 joints
Joints:
- joint joint2: axis 0 0 1 -> 0 0 -1
- joint joint3: axis 0 0 1 -> 0 0 -1
- joint joint4: origin xyz=0 0.012 0.054 rpy=-1.5708 0 0 -> xyz=0 0.012 0.054 rpy=1.5708 0 3.1416

Commit message: feat: 现实验证完成

File: src/arm_description/urdf/miniarm.urdf (robot description, URDF)
Before this commit: robot mini1, 7 links, 6 joints
Joints:
- joint joint2: axis 0 0 -1 -> 0 0 1
- joint joint3: axis 0 0 -1 -> 0 0 1
- joint joint4: axis 0 0 -1 -> 0 0 1
- joint joint6: axis 0 0 -1 -> 0 0 1

Commit message: feat: 末端伺服真实情况验证完毕

File: src/arm_description/urdf/miniarm.urdf (robot description, URDF)
Before this commit: robot mini1, 7 links, 6 joints
Joints:
- joint joint3: limit lower=-0.785398 upper=1.1570796 effort=9.0 velocity=18.0 -> lower=-2.7925 upper=0.1 effort=9.0 velocity=18.0
- joint joint4: limit lower=-3.1415926535 upper=3.1415926535 effort=3.5 velocity=18.0 -> lower=-1.57 upper=1.57 effort=3.5 velocity=18.0
